File: hardware/swadge-devkit.sch (KiCad schematic (older format))
At the start: 1 part, among them U1 ESP-12F

Commit message: Worked on the schematic
Added accelerometer part lib
Parts:
- added BT1: Battery, Battery:BatteryHolder_MPD_BC2AAPC_2xAA, symbol Device:Battery
- added C1: 22u, Capacitor_SMD:C_0603_1608Metric, symbol Device:C
- added C10, C11, C4, C5, C6, C7, C8, C9: 1u, Capacitor_SMD:C_0603_1608Metric, symbol Device:C
- added C12, C14: 0.1u, Capacitor_SMD:C_0603_1608Metric, symbol Device:C
- added C13: 4.7u, Capacitor_SMD:C_0603_1608Metric, symbol Device:C
- added C2, C3: 0.22u, Capacitor_SMD:C_0603_1608Metric, symbol Device:C
- added D1, D2, D3, D4, D5, D6, D7, D8: WS2812B, LED_SMD:LED_WS2812B_PLCC4_5.0x5.0mm_P3.2mm, symbol LED:WS2812B
- added J1: USB_B_Micro, Connector_USB:USB_Micro-B_Molex_47346-0001, symbol Connector:USB_B_Micro
- added MK1: Microphone, Capacitor_THT:CP_Radial_D8.0mm_P3.80mm, symbol Device:Microphone
- added R1: 1K, Resistor_SMD:R_0603_1608Metric, symbol Device:R_US
- added R10, R11, R3, R5, R6, R9: 10K, Resistor_SMD:R_0603_1608Metric, symbol Device:R_US
- added R12, R13: 10k, Resistor_SMD:R_0603_1608Metric, symbol Device:R_US
- added R2, R4: 47K, Resistor_SMD:R_0603_1608Metric, symbol Device:R_US
- added R7: 220K, Resistor_SMD:R_0603_1608Metric, symbol Device:R_US
- added R8: 70, Resistor_SMD:R_0603_1608Metric, symbol Device:R_US
- added SW1: SW_SPDT, Button_Switch_SMD:SW_SPDT_CK-JS102011SAQN, symbol Switch:SW_SPDT
- added SW2, SW3, SW4, SW5: SW_Push, Button_Switch_SMD:SW_SPST_B3S-1000, symbol Switch:SW_Push
- added U2: MCP6001-OT, Package_TO_SOT_SMD:SOT-23-5, symbol Amplifier_Operational:MCP6001-OT
- added U3: MMA8452Q, MMA8452Q:QFN-16_0.5MM, symbol MMA8452Q:MMA8452Q
- added U4: AP1117-33, Package_TO_SOT_SMD:SOT-223-3_TabPin2, symbol Regulator_Linear:AP1117-33
Connections:
- net labels added: +3.3V, ADC_PIN, AUD_PWR, GND, GPIO0, GPIO10, GPIO12, GPIO13, GPIO15, GPIO16, GPIO2, RX, SCL, SDA, TX
- wire segments 0 -> 78
- no-connect marks 0 -> 5
Other:
- note added: "Accelerometer Circuit"
- note added: "Boot Resistors"
- note added: "Buttons"
- note added: "ESP8266 Circuit"
- note added: "GPIO0 is pulled high to boot\nnormally and low to enter\nUART programming mode"
- note added: "If GPIO2 is low and GPIO15\nis high it will boot in\nSD-Card mode"
- note added: "LED Circuit"
- note added: "Microphone Circuit"
- note added: "Power Circuit"
- note added: "TODO: Display\nTODO: M.2 Connector\nTODO: Bypass Caps"

Commit message: Added PCIE connector
Parts:
- added U5: BUS_PCIexpress, Connector_PCBEdge:BUS_PCIexpress, symbol Connector_PCBEdge:BUS_PCIexpress
Connections:
- net labels added: +5V, CS0, MISO, MOSI, REST, SCLK, SW2, SW3, SW4, SW5
- net labels removed: GPIO10, GPIO12, GPIO13, GPIO16
- wire segments 78 -> 96
Other:
- note added: "Edge Connector"
- note added: "TODO: Display\nTODO: Bypass Caps"
- note removed: "TODO: Display\nTODO: M.2 Connector\nTODO: Bypass Caps"
Changed lines of the file:
@@
 L power:+3.3V #PWR0103
 U 1 1 5C3B284C
-P 650 3750
-F 0 "#PWR0103" H 650 3600 50  0001 C CNN
-F 1 "+3.3V" H 665 3923 50  0000 C CNN
-F 2 "" H 650 3750 50  0001 C CNN
-F 3 "" H 650 3750 50  0001 C CNN
-	1    650  3750
+P 600 3250
+F 0 "#PWR0103" H 600 3100 50  0001 C CNN
+F 1 "+3.3V" H 615 3423 50  0000 C CNN
+F 2 "" H 600 3250 50  0001 C CNN
+F 3 "" H 600 3250 50  0001 C CNN
+	1    600  3250
 	1    0    0    -1
 $EndComp
 Text GLabel 2100 4250 3    50   Input ~ 0
-GPIO10
+SW2
 Text GLabel 2950 3650 2    50   Input ~ 0
 GPIO15
@@
 	1150 4850 1150 4700
 Text Notes 5850 2800 0    50   ~ 0
-TODO: Display\nTODO: M.2 Connector\nTODO: Bypass Caps
+TODO: Display\nTODO: Bypass Caps
 $Comp
 L Regulator_Linear:AP1117-33 U4
 U 1 1 5C3ED77E
-P 10150 1500
-F 0 "U4" H 10150 1742 50  0000 C CNN
-F 1 "AP1117-33" H 10150 1651 50  0000 C CNN
-F 2 "Package_TO_SOT_SMD:SOT-223-3_TabPin2" H 10150 1700 50  0001 C CNN
-F 3 "http://www.diodes.com/datasheets/AP1117.pdf" H 10250 1250 50  0001 C CNN
-	1    10150 1500
+P 10150 1700
+F 0 "U4" H 10150 1942 50  0000 C CNN
+F 1 "AP1117-33" H 10150 1851 50  0000 C CNN
+F 2 "Package_TO_SOT_SMD:SOT-223-3_TabPin2" H 10150 1900 50  0001 C CNN
+F 3 "http://www.diodes.com/datasheets/AP1117.pdf" H 10250 1450 50  0001 C CNN
+	1    10150 1700
 	1    0    0    -1
 $EndComp
@@
 	-1   0    0    1
 $EndComp
-Wire Wire Line
-	9800 1500 9850 1500
-Wire Wire Line
-	10150 1800 10150 2100
-Wire Wire Line
-	10150 2100 9850 2100
 Connection ~ 9500 2100
 $Comp
@@
 	1    0    0    -1
 $EndComp
-Connection ~ 9850 2100
 Wire Wire Line
 	9850 2100 9500 2100
@@
 Wire Wire Line
 	10450 1050 10450 1200
-Wire Wire Line
-	10450 1400 10450 1500
 Wire Wire Line
 	10850 1300 11000 1300
@@
 Text GLabel 2950 3350 2    50   Input ~ 0
 SDA
-Wire Wire Line
-	1150 3750 650  3750
 Text GLabel 4150 3300 0    50   Input ~ 0
-GPIO10
+SW2
 Text GLabel 1150 3550 0    50   Input ~ 0
-GPIO12
+SW4
 Text GLabel 1150 3650 0    50   Input ~ 0
-GPIO13
-Text GLabel 1150 3350 0    50   Input ~ 0
-GPIO16
+SW3
 Text GLabel 5100 3850 0    50   Input ~ 0
-GPIO16
+SW5
 Text GLabel 5100 3300 0    50   Input ~ 0
-GPIO12
+SW4
 Text GLabel 4150 3850 0    50   Input ~ 0
-GPIO13
+SW3
 $Comp
 L Switch:SW_Push SW2
@@
 Wire Wire Line
 	1000 850  1350 850
+$Comp
+L Connector_PCBEdge:BUS_PCIexpress U5
+U 1 1 5C3B5040
+P 4700 6250
+F 0 "U5" H 4700 7325 50  0000 C CNN
+F 1 "BUS_PCIexpress" H 4700 7234 50  0000 C CNN
+F 2 "Connector_PCBEdge:BUS_PCIexpress" H 4700 6600 50  0001 C CNN
+F 3 "https://www.digikey.com/products/en/connectors-interconnects/card-edge-connectors-edgeboard-connectors/303?FV=1600024%2C85c0002%2C1f140000%2Cffe0012f&quantity=0&ColumnSort=1000011&page=1&stock=1&pageSize=25" H 4700 6600 50  0001 C CNN
+	1    4700 6250
+	1    0    0    -1
+$EndComp
+Text GLabel 1100 3050 1    50   Input ~ 0
+REST
+Text GLabel 4500 5400 0    50   Input ~ 0
+REST
+Text GLabel 4900 5400 2    50   Input ~ 0
+ADC_PIN
+Text GLabel 4500 5600 0    50   Input ~ 0
+AUD_PWR
+Text GLabel 4900 5600 2    50   Input ~ 0
+SW4
+Text GLabel 4500 6400 0    50   Input ~ 0
+SW3
+$Comp
+L power:+3.3V #PWR0110
+U 1 1 5C3B6600
+P 5000 6200
+F 0 "#PWR0110" H 5000 6050 50  0001 C CNN
+F 1 "+3.3V" H 5015 6373 50  0000 C CNN
+F 2 "" H 5000 6200 50  0001 C CNN
+F 3 "" H 5000 6200 50  0001 C CNN
+	1    5000 6200
+	1    0    0    -1
+$EndComp
+Text GLabel 1800 4250 3    50   Input ~ 0
+CS0
+Text GLabel 1900 4250 3    50   Input ~ 0
+MISO
+Text GLabel 2000 4250 3    50   Input ~ 0
+SW5
+Text GLabel 2200 4250 3    50   Input ~ 0
+MOSI
+Text GLabel 2300 4250 3    50   Input ~ 0
+SCLK
+Text GLabel 4500 6500 0    50   Input ~ 0
+CS0
+Text GLabel 4900 6400 2    50   Input ~ 0
+MISO
+Text GLabel 4500 6600 0    50   Input ~ 0
+SW5
+Text GLabel 4900 6500 2    50   Input ~ 0
+SW2
+Text GLabel 4500 6800 0    50   Input ~ 0
+MOSI
+Text GLabel 4900 6600 2    50   Input ~ 0
+SCLK
+Text GLabel 4900 6800 2    50   Input ~ 0
+GPIO15
+Text GLabel 4900 6900 2    50   Input ~ 0
+GPIO0
+Text GLabel 4900 7000 2    50   Input ~ 0
+SCL
+Text GLabel 4900 7100 2    50   Input ~ 0
+TX
+Text GLabel 4500 6900 0    50   Input ~ 0
+GPIO2
+Text GLabel 4500 7000 0    50   Input ~ 0
+SDA
+Text GLabel 4500 7100 0    50   Input ~ 0
+RX
+$Comp
+L power:GND #PWR0111
+U 1 1 5C3BA3DC
+P 4300 6000
+F 0 "#PWR0111" H 4300 5750 50  0001 C CNN
+F 1 "GND" H 4305 5827 50  0000 C CNN
+F 2 "" H 4300 6000 50  0001 C CNN
+F 3 "" H 4300 6000 50  0001 C CNN
+	1    4300 6000
+	1    0    0    -1
+$EndComp
+$Comp
+L power:+5V #PWR038
+U 1 1 5C3BE999
+P 9900 1500
+F 0 "#PWR038" H 9900 1350 50  0001 C CNN
+F 1 "+5V" H 9915 1673 50  0000 C CNN
+F 2 "" H 9900 1500 50  0001 C CNN
+F 3 "" H 9900 1500 50  0001 C CNN
+	1    9900 1500
+	1    0    0    -1
+$EndComp
+Wire Wire Line
+	9800 1500 9850 1500
+Connection ~ 9850 1500
+Wire Wire Line
+	9850 1500 9900 1500
+Wire Wire Line
+	10150 2100 9850 2100
+Connection ~ 9850 2100
+Wire Wire Line
+	10450 1700 10450 1400
+Wire Wire Line
+	9850 1700 9850 1500
+Wire Wire Line
+	10150 2000 10150 2100
+$Comp
+L power:+5V #PWR037
+U 1 1 5C3CDED6
+P 5000 5900
+F 0 "#PWR037" H 5000 5750 50  0001 C CNN
+F 1 "+5V" H 5015 6073 50  0000 C CNN
+F 2 "" H 5000 5900 50  0001 C CNN
+F 3 "" H 5000 5900 50  0001 C CNN
+	1    5000 5900
+	1    0    0    -1
+$EndComp
+Wire Wire Line
+	4900 5800 4900 5900
+Wire Wire Line
+	5000 5900 4900 5900
+Connection ~ 4900 5900
+Wire Wire Line
+	4900 6100 4900 6200
+Wire Wire Line
+	4900 6200 5000 6200
+Connection ~ 4900 6200
+Wire Wire Line
+	4500 5800 4500 5900
+Wire Wire Line
+	4500 5900 4500 6000
+Connection ~ 4500 5900
+Wire Wire Line
+	4500 6000 4500 6100
+Connection ~ 4500 6000
+Wire Wire Line
+	4500 6100 4500 6200
+Connection ~ 4500 6100
+Wire Wire Line
+	4300 6000 4500 6000
+Wire Notes Line
+	3700 4700 3700 7750
+Wire Notes Line
+	3700 7750 5700 7750
+Wire Notes Line
+	5700 7750 5700 4700
+Wire Notes Line
+	5700 4700 3700 4700
+Text Notes 3750 4800 0    50   ~ 0
+Edge Connector
+Wire Notes Line
+	3700 4850 4400 4850
+Wire Notes Line
+	4400 4850 4400 4700
+Wire Wire Line
+	4500 5500 4500 5400
+Wire Wire Line
+	1150 3750 600  3750
+Wire Wire Line
+	600  3750 600  3250
+Wire Wire Line
+	1150 3250 600  3250
+Connection ~ 600  3250
+Wire Wire Line
+	1150 3350 750  3350
+Wire Wire Line
+	750  3350 750  3050
+Wire Wire Line
+	750  3050 1100 3050
+Connection ~ 1100 3050
+Wire Wire Line
+	1100 3050 1150 3050
 $EndSCHEMATC

Commit message: Routed everything
Connections:
- wire segments 96 -> 170
- no-connect marks 5 -> 18

Commit message: Added I2C display
Schematic copied from https://github.com/adafruit/Adafruit-1.3inch-128x64-Mono-OLED-PCB
Parts:
- added C15, C16, C17, C18, C19: 2.2u, Capacitor_SMD:C_0603_1608Metric, symbol Device:C
- added C20: 10u, Capacitor_SMD:C_0603_1608Metric, symbol Device:C
- added R14: 390k, Resistor_SMD:R_0603_1608Metric, symbol Device:R_US
- added U6: DISP_OLED_UG-2864HSWEG01, disp_oled:microbuilder-UG-2864HSWEG01_1.3_WRAPAROUND, symbol disp_oled:DISP_OLED_UG-2864HSWEG01
- C12: value 0.1u -> 4.7u
- C13: value 4.7u -> 0.1u
Connections:
- wire segments 170 -> 214
- no-connect marks 18 -> 27
Other:
- note added: "10k pullups are in the\naccelerometer section"
- note added: "Display Circuit"
- note added: "I2C Address 0x78\nw/ SA0 at GND"
- note added: "I2C address 0x1C\nw/SA0 at GND"
- note added: "TODO: Bypass Caps\nTODO: ESP-12F GND on bottom?"
- note removed: "TODO: Display\nTODO: Bypass Caps"

Commit message: Updated power switch
Parts:
- SW1: footprint Button_Switch_SMD:SW_SPDT_CK-JS102011SAQN -> Button_Switch_SMD:SW_SPDT_PCM12
Changed lines of the file:
@@
 EESchema Schematic File Version 4
-LIBS:swadge-devkit-cache
 EELAYER 26 0
 EELAYER END
@@
 F 0 "SW1" H 10800 1950 50  0000 C CNN
 F 1 "SW_SPDT" H 10800 1850 50  0000 C CNN
-F 2 "Button_Switch_SMD:SW_SPDT_CK-JS102011SAQN" H 10800 1650 50  0001 C CNN
+F 2 "Button_Switch_SMD:SW_SPDT_PCM12" H 10800 1650 50  0001 C CNN
 F 3 "" H 10800 1650 50  0001 C CNN
 	1    10800 1650

Commit message: Added more 3D parts!
Parts:
- removed BT1: Battery, Battery:BatteryHolder_MPD_BC2AAPC_2xAA, symbol Device:Battery
- removed SW2, SW3, SW4, SW5: SW_Push, Button_Switch_SMD:SW_SPST_B3S-1000, symbol Switch:SW_Push
- added SW2, SW3, SW4, SW5: 4-1437565-2, 4-1437565-2:SW_4-1437565-2, symbol 4-1437565-2:4-1437565-2
- added U7, U8: 2460, SamacSys_Parts:2460, symbol SamacSys_Parts:2460
Connections:
- wire segments 214 -> 228

Commit message: Made a new microphone footprint, added 3D microphone model
Parts:
- MK1: footprint Capacitor_THT:CP_Radial_D8.0mm_P3.80mm -> microphone:POM-2738P-R
Changed lines of the file:
@@
 F 0 "MK1" H 2280 2046 50  0000 L CNN
 F 1 "Microphone" H 2280 1955 50  0000 L CNN
-F 2 "Capacitor_THT:CP_Radial_D8.0mm_P3.80mm" V 2150 2100 50  0001 C CNN
+F 2 "microphone:POM-2738P-R" V 2150 2100 50  0001 C CNN
 F 3 "~" V 2150 2100 50  0001 C CNN
 	1    2150 2000
