File: hardware/swadge-programmer.sch (KiCad schematic (older format))
At the start: 14 parts, among them J1 USB_B_Micro, SW1 SW_Push_SPDT, SW2 SW_Push_SPDT, SW3 SW_Push_SPDT, U1 BUS_PCIexpress, U2 CP2102N-A01-GQFN24

Commit message: Added power switches & pin headers to programmer
Parts:
- added J2: Conn_02x21_Top_Bottom, Connector_PinHeader_2.54mm:PinHeader_2x21_P2.54mm_Vertical, symbol Connector_Generic:Conn_02x21_Top_Bottom
- added SW4, SW5: SW_DPDT_x2, JS202011CQN:JS202011CQN, symbol Switch:SW_DPDT_x2
Connections:
- net labels added: 3.3V, 5V
- wire segments 79 -> 126
- no-connect marks 15 -> 19
Other:
- note added: "Connectors"
- note added: "GPIO Switches"
- note added: "Power Switches"
- note added: "USB to UART"

Commit message: Started updating programmer to use local parts
Parts:
- C1, C2, C3, C4: footprint Capacitor_SMD:C_0603_1608Metric -> Swadge_Parts:C_0603_1608Metric; symbol Device:C -> Swadge_Parts:C
- J1: footprint Connector_USB:USB_Micro-B_Molex_47346-0001 -> Swadge_Parts:USB_Micro-B_Molex_47346-0001; symbol Connector:USB_B_Micro -> Swadge_Parts:USB_B_Micro
- R1, R2, R3: footprint Resistor_SMD:R_0603_1608Metric -> Swadge_Parts:R_0603_1608Metric; symbol Device:R_US -> Swadge_Parts:R_US
- SW4, SW5: footprint JS202011CQN:JS202011CQN -> Swadge_Parts:JS202011CQN; symbol Switch:SW_DPDT_x2 -> Swadge_Parts:SW_DPDT_x2
- U1: footprint 10018784-10210TLF:10018784-10210TLF -> Swadge_Parts:10018784-10210TLF; symbol Connector_PCBEdge:BUS_PCIexpress -> Swadge_Parts:BUS_PCIexpress
Changed lines of the file:
@@
 $EndComp
 $Comp
-L Connector_PCBEdge:BUS_PCIexpress U1
+L Swadge_Parts:BUS_PCIexpress U1
 U 1 1 5C4297AA
 P 1200 4950
 F 0 "U1" H 1200 6025 50  0000 C CNN
 F 1 "BUS_PCIexpress" H 1200 5934 50  0000 C CNN
-F 2 "10018784-10210TLF:10018784-10210TLF" H 1200 5300 50  0001 C CNN
+F 2 "Swadge_Parts:10018784-10210TLF" H 1200 5300 50  0001 C CNN
 F 3 "" H 1200 5300 50  0001 C CNN
 	1    1200 4950
@@
 	3750 2050 3800 2050
 $Comp
-L Connector:USB_B_Micro J1
+L Swadge_Parts:USB_B_Micro J1
 U 1 1 5C43540A
 P 800 2650
 F 0 "J1" H 855 3117 50  0000 C CNN
 F 1 "USB_B_Micro" H 855 3026 50  0000 C CNN
-F 2 "Connector_USB:USB_Micro-B_Molex_47346-0001" H 950 2600 50  0001 C CNN
+F 2 "Swadge_Parts:USB_Micro-B_Molex_47346-0001" H 950 2600 50  0001 C CNN
 F 3 "~" H 950 2600 50  0001 C CNN
 	1    800  2650
@@
 Connection ~ 1200 3300
 $Comp
-L Device:R_US R1
+L Swadge_Parts:R_US R1
 U 1 1 5C444907
 P 1300 1800
 F 0 "R1" H 1368 1846 50  0000 L CNN
 F 1 "22.1k" H 1368 1755 50  0000 L CNN
-F 2 "Resistor_SMD:R_0603_1608Metric" V 1340 1790 50  0001 C CNN
+F 2 "Swadge_Parts:R_0603_1608Metric" V 1340 1790 50  0001 C CNN
 F 3 "~" H 1300 1800 50  0001 C CNN
 	1    1300 1800
@@
 $EndComp
 $Comp
-L Device:R_US R2
+L Swadge_Parts:R_US R2
 U 1 1 5C444A33
 P 1300 2200
 F 0 "R2" H 1368 2246 50  0000 L CNN
 F 1 "47.5k" H 1368 2155 50  0000 L CNN
-F 2 "Resistor_SMD:R_0603_1608Metric" V 1340 2190 50  0001 C CNN
+F 2 "Swadge_Parts:R_0603_1608Metric" V 1340 2190 50  0001 C CNN
 F 3 "~" H 1300 2200 50  0001 C CNN
 	1    1300 2200
@@
 Connection ~ 1300 3300
 $Comp
-L Device:R_US R3
+L Swadge_Parts:R_US R3
 U 1 1 5C465A56
 P 2550 1250
 F 0 "R3" H 2482 1204 50  0000 R CNN
 F 1 "1k" H 2482 1295 50  0000 R CNN
-F 2 "Resistor_SMD:R_0603_1608Metric" V 2590 1240 50  0001 C CNN
+F 2 "Swadge_Parts:R_0603_1608Metric" V 2590 1240 50  0001 C CNN
 F 3 "~" H 2550 1250 50  0001 C CNN
 	1    2550 1250
@@
 $EndComp
 $Comp
-L Device:C C4
+L Swadge_Parts:C C4
 U 1 1 5C473CF2
 P 2150 1800
 F 0 "C4" H 2265 1846 50  0000 L CNN
 F 1 "4.7u" H 2265 1755 50  0000 L CNN
-F 2 "Capacitor_SMD:C_0603_1608Metric" H 2188 1650 50  0001 C CNN
+F 2 "Swadge_Parts:C_0603_1608Metric" H 2188 1650 50  0001 C CNN
 F 3 "~" H 2150 1800 50  0001 C CNN
 	1    2150 1800
@@
 $EndComp
 $Comp
-L Device:C C3
+L Swadge_Parts:C C3
 U 1 1 5C473DAA
 P 1750 1800
 F 0 "C3" H 1865 1846 50  0000 L CNN
 F 1 "0.1u" H 1865 1755 50  0000 L CNN
-F 2 "Capacitor_SMD:C_0603_1608Metric" H 1788 1650 50  0001 C CNN
+F 2 "Swadge_Parts:C_0603_1608Metric" H 1788 1650 50  0001 C CNN
 F 3 "~" H 1750 1800 50  0001 C CNN
 	1    1750 1800
@@
 $EndComp
 $Comp
-L Device:C C2
+L Swadge_Parts:C C2
 U 1 1 5C473DE0
 P 3750 1000
 F 0 "C2" H 3865 1046 50  0000 L CNN
 F 1 "4.7u" H 3865 955 50  0000 L CNN
-F 2 "Capacitor_SMD:C_0603_1608Metric" H 3788 850 50  0001 C CNN
+F 2 "Swadge_Parts:C_0603_1608Metric" H 3788 850 50  0001 C CNN
 F 3 "~" H 3750 1000 50  0001 C CNN
 	1    3750 1000
@@
 $EndComp
 $Comp
-L Device:C C1
+L Swadge_Parts:C C1
 U 1 1 5C473E18
 P 3300 1000
 F 0 "C1" H 3415 1046 50  0000 L CNN
 F 1 "0.1u" H 3415 955 50  0000 L CNN
-F 2 "Capacitor_SMD:C_0603_1608Metric" H 3338 850 50  0001 C CNN
+F 2 "Swadge_Parts:C_0603_1608Metric" H 3338 850 50  0001 C CNN
 F 3 "~" H 3300 1000 50  0001 C CNN
 	1    3300 1000
@@
 Connection ~ 3050 5950
 $Comp
-L Switch:SW_DPDT_x2 SW4
+L Swadge_Parts:SW_DPDT_x2 SW4
 U 1 1 5C4F30A9
 P 4800 1000
 F 0 "SW4" H 4800 1285 50  0000 C CNN
 F 1 "SW_DPDT_x2" H 4800 1194 50  0000 C CNN
-F 2 "JS202011CQN:JS202011CQN" H 4800 1000 50  0001 C CNN
+F 2 "Swadge_Parts:JS202011CQN" H 4800 1000 50  0001 C CNN
 F 3 "" H 4800 1000 50  0001 C CNN
 	1    4800 1000
@@
 $EndComp
 $Comp
-L Switch:SW_DPDT_x2 SW4
+L Swadge_Parts:SW_DPDT_x2 SW4
 U 2 1 5C4F314E
 P 4800 1550
 F 0 "SW4" H 4800 1835 50  0000 C CNN
 F 1 "SW_DPDT_x2" H 4800 1744 50  0000 C CNN
-F 2 "JS202011CQN:JS202011CQN" H 4800 1550 50  0001 C CNN
+F 2 "Swadge_Parts:JS202011CQN" H 4800 1550 50  0001 C CNN
 F 3 "" H 4800 1550 50  0001 C CNN
 	2    4800 1550
@@
 $EndComp
 $Comp
-L Switch:SW_DPDT_x2 SW5
+L Swadge_Parts:SW_DPDT_x2 SW5
 U 2 1 5C48B8E0
 P 5500 900
 F 0 "SW5" H 5500 1185 50  0000 C CNN
 F 1 "SW_DPDT_x2" H 5500 1094 50  0000 C CNN
-F 2 "JS202011CQN:JS202011CQN" H 5500 900 50  0001 C CNN
+F 2 "Swadge_Parts:JS202011CQN" H 5500 900 50  0001 C CNN
 F 3 "" H 5500 900 50  0001 C CNN
 	2    5500 900
@@
 $EndComp
 $Comp
-L Switch:SW_DPDT_x2 SW5
+L Swadge_Parts:SW_DPDT_x2 SW5
 U 1 1 5C48B922
 P 5450 1650
 F 0 "SW5" H 5450 1935 50  0000 C CNN
 F 1 "SW_DPDT_x2" H 5450 1844 50  0000 C CNN
-F 2 "JS202011CQN:JS202011CQN" H 5450 1650 50  0001 C CNN
+F 2 "Swadge_Parts:JS202011CQN" H 5450 1650 50  0001 C CNN
 F 3 "" H 5450 1650 50  0001 C CNN
 	1    5450 1650

Commit message: Moved all programmer parts into this repo
Resized programmer, rerouted programmer, added holes
Parts:
- removed SW1, SW2, SW3: SW_Push_SPDT, Button_Switch_SMD:SW_SPDT_PCM12, symbol Switch:SW_Push_SPDT
- added H1, H2, H3, H4: Hole, Swadge_Parts:Hole, symbol Swadge_Parts:Hole
- added J3: Conn_02x21_Top_Bottom, Swadge_Parts:PinHeader_2x21_P2.54mm_Vertical, symbol Swadge_Parts:Conn_02x21_Top_Bottom
- added R4, R5: 1, Swadge_Parts:R_Axial_DIN0207_L6.3mm_D2.5mm_P10.16mm_Horizontal, symbol Swadge_Parts:R_US
- added SW1, SW2, SW3: SW_DPDT_x2, Swadge_Parts:JS202011CQN, symbol Swadge_Parts:SW_DPDT_x2
- D1: footprint Package_TO_SOT_SMD:SOT-143 -> Swadge_Parts:SOT-143; symbol Power_Protection:SP0503BAHT -> Swadge_Parts:SP0503BAHT
- J2: footprint Connector_PinHeader_2.54mm:PinHeader_2x21_P2.54mm_Vertical -> Swadge_Parts:PinHeader_2x21_P2.54mm_Vertical; symbol Connector_Generic:Conn_02x21_Top_Bottom -> Swadge_Parts:Conn_02x21_Top_Bottom
- U2: footprint Package_DFN_QFN:QFN-24-1EP_4x4mm_P0.5mm_EP2.6x2.6mm -> Swadge_Parts:QFN-24-1EP_4x4mm_P0.5mm_EP2.6x2.6mm; symbol Interface_USB:CP2102N-A01-GQFN24 -> Swadge_Parts:CP2102N-A01-GQFN24
Connections:
- wire segments 126 -> 172
Other:
- note added: "Holes"

Commit message: Updated programmer traces, parts, BOM
Parts:
- C1, C2, C3, C4, R1, R2, R3, R4, R5: Cost100 (none) -> 10; Digikey (none) -> n/a; Substitutable (none) -> Y
- D1: Cost100 (none) -> 95; Digikey (none) -> F2715CT-ND; Substitutable (none) -> Y
- H1, H2, H3, H4, U1: Cost100 (none) -> 0; Digikey (none) -> n/a; NOBOM (none) -> y; Substitutable (none) -> Y
- J1: Cost100 (none) -> 112; Digikey (none) -> WM17141CT-ND; Substitutable (none) -> Y
- J2, J3: Cost100 (none) -> 73; Digikey (none) -> S2012EC-21-ND; Substitutable (none) -> Y
- SW1, SW2, SW3, SW4, SW5: Cost100 (none) -> 45; Digikey (none) -> 401-2001-ND; Substitutable (none) -> Y
- U2: Cost100 (none) -> 135; Digikey (none) -> 336-4737-1-ND; Substitutable (none) -> Y

Commit message: Updated digikey part numbers Added graphics to swadge programmer PCB
Parts:
- C1, C3: Digikey n/a -> 1276-1000-1-ND
- C2, C4: Digikey n/a -> 1276-1045-1-ND
- R1: Digikey n/a -> RMCF0603FT22K1CT-ND
- R2: Digikey n/a -> P47.5KHCT-ND
- R3: Digikey n/a -> RMCF0603FT1K00DKR-ND
- R4, R5: Digikey n/a -> RNF14FTD1R00CT-ND
Changed lines of the file:
@@
 F 3 "" H 1300 1800 50  0001 C CNN
 F 4 "10" H 0   0   50  0001 C CNN "Cost100"
-F 5 "n/a" H 0   0   50  0001 C CNN "Digikey"
+F 5 "RMCF0603FT22K1CT-ND" H 0   0   50  0001 C CNN "Digikey"
 F 6 "Y" H 0   0   50  0001 C CNN "Substitutable"
 	1    1300 1800
@@
 F 3 "" H 1300 2200 50  0001 C CNN
 F 4 "10" H 0   0   50  0001 C CNN "Cost100"
-F 5 "n/a" H 0   0   50  0001 C CNN "Digikey"
+F 5 "P47.5KHCT-ND" H 0   0   50  0001 C CNN "Digikey"
 F 6 "Y" H 0   0   50  0001 C CNN "Substitutable"
 	1    1300 2200
@@
 F 3 "" H 2550 1250 50  0001 C CNN
 F 4 "10" H 0   0   50  0001 C CNN "Cost100"
-F 5 "n/a" H 0   0   50  0001 C CNN "Digikey"
+F 5 "RMCF0603FT1K00DKR-ND" H 0   0   50  0001 C CNN "Digikey"
 F 6 "Y" H 0   0   50  0001 C CNN "Substitutable"
 	1    2550 1250
@@
 F 3 "" H 2150 1800 50  0001 C CNN
 F 4 "10" H 0   0   50  0001 C CNN "Cost100"
-F 5 "n/a" H 0   0   50  0001 C CNN "Digikey"
+F 5 "1276-1045-1-ND" H 0   0   50  0001 C CNN "Digikey"
 F 6 "Y" H 0   0   50  0001 C CNN "Substitutable"
 	1    2150 1800
@@
 F 3 "" H 1750 1800 50  0001 C CNN
 F 4 "10" H 0   0   50  0001 C CNN "Cost100"
-F 5 "n/a" H 0   0   50  0001 C CNN "Digikey"
+F 5 "1276-1000-1-ND" H 0   0   50  0001 C CNN "Digikey"
 F 6 "Y" H 0   0   50  0001 C CNN "Substitutable"
 	1    1750 1800
@@
 F 3 "" H 3750 1000 50  0001 C CNN
 F 4 "10" H 0   0   50  0001 C CNN "Cost100"
-F 5 "n/a" H 0   0   50  0001 C CNN "Digikey"
+F 5 "1276-1045-1-ND" H 0   0   50  0001 C CNN "Digikey"
 F 6 "Y" H 0   0   50  0001 C CNN "Substitutable"
 	1    3750 1000
@@
 F 3 "" H 3300 1000 50  0001 C CNN
 F 4 "10" H 0   0   50  0001 C CNN "Cost100"
-F 5 "n/a" H 0   0   50  0001 C CNN "Digikey"
+F 5 "1276-1000-1-ND" H 0   0   50  0001 C CNN "Digikey"
 F 6 "Y" H 0   0   50  0001 C CNN "Substitutable"
 	1    3300 1000
@@
 F 3 "" H 1600 4100 50  0001 C CNN
 F 4 "10" H 0   0   50  0001 C CNN "Cost100"
-F 5 "n/a" H 0   0   50  0001 C CNN "Digikey"
+F 5 "RNF14FTD1R00CT-ND" H 0   0   50  0001 C CNN "Digikey"
 F 6 "Y" H 0   0   50  0001 C CNN "Substitutable"
 	1    1600 4100
@@
 F 3 "" H 1600 5200 50  0001 C CNN
 F 4 "10" H 0   0   50  0001 C CNN "Cost100"
-F 5 "n/a" H 0   0   50  0001 C CNN "Digikey"
+F 5 "RNF14FTD1R00CT-ND" H 0   0   50  0001 C CNN "Digikey"
 F 6 "Y" H 0   0   50  0001 C CNN "Substitutable"
 	1    1600 5200

Commit message: Updated digikey part numbers
Parts:
- R3: Digikey RMCF0603FT1K00DKR-ND -> 311-1.00KHRCT-ND
Changed lines of the file:
@@
 F 3 "" H 2550 1250 50  0001 C CNN
 F 4 "10" H 0   0   50  0001 C CNN "Cost100"
-F 5 "RMCF0603FT1K00DKR-ND" H 0   0   50  0001 C CNN "Digikey"
+F 5 "311-1.00KHRCT-ND" H 0   0   50  0001 C CNN "Digikey"
 F 6 "Y" H 0   0   50  0001 C CNN "Substitutable"
 	1    2550 1250

Commit message: #16 replace GPIO switches with buttons in schematic
Parts:
- removed SW1, SW2, SW3: SW_DPDT_x2, Swadge_Parts:JS202011CQN, symbol Swadge_Parts:SW_DPDT_x2
- added SW1, SW2, SW3: 4-1437565-2, Swadge_Parts:SW_4-1437565-2, symbol Swadge_Parts:4-1437565-2
Connections:
- wire segments 172 -> 178
- no-connect marks 19 -> 16
Changed lines of the file:
@@
 EESchema Schematic File Version 4
-LIBS:swadge-programmer-cache
 EELAYER 26 0
 EELAYER END
@@
 Text GLabel 6500 2300 0    50   Input ~ 0
 GPIO15
-NoConn ~ 6950 900
-NoConn ~ 6950 1550
-NoConn ~ 6950 2200
 $Comp
 L power:GND #PWR05
 U 1 1 5C42F52E
-P 7100 1150
-F 0 "#PWR05" H 7100 900 50  0001 C CNN
-F 1 "GND" H 7105 977 50  0000 C CNN
-F 2 "" H 7100 1150 50  0001 C CNN
-F 3 "" H 7100 1150 50  0001 C CNN
-	1    7100 1150
+P 7200 1050
+F 0 "#PWR05" H 7200 800 50  0001 C CNN
+F 1 "GND" H 7205 877 50  0000 C CNN
+F 2 "" H 7200 1050 50  0001 C CNN
+F 3 "" H 7200 1050 50  0001 C CNN
+	1    7200 1050
 	1    0    0    -1
 $EndComp
@@
 L power:GND #PWR06
 U 1 1 5C42F541
-P 7100 1800
-F 0 "#PWR06" H 7100 1550 50  0001 C CNN
-F 1 "GND" H 7105 1627 50  0000 C CNN
-F 2 "" H 7100 1800 50  0001 C CNN
-F 3 "" H 7100 1800 50  0001 C CNN
-	1    7100 1800
-	1    0    0    -1
-$EndComp
-Wire Wire Line
-	6950 1750 7100 1750
-Wire Wire Line
-	7100 1750 7100 1800
-Wire Wire Line
-	6950 1100 7100 1100
-Wire Wire Line
-	7100 1100 7100 1150
+P 7200 1700
+F 0 "#PWR06" H 7200 1450 50  0001 C CNN
+F 1 "GND" H 7205 1527 50  0000 C CNN
+F 2 "" H 7200 1700 50  0001 C CNN
+F 3 "" H 7200 1700 50  0001 C CNN
+	1    7200 1700
+	1    0    0    -1
+$EndComp
+Wire Wire Line
+	7050 1650 7200 1650
+Wire Wire Line
+	7200 1650 7200 1700
+Wire Wire Line
+	7050 1000 7200 1000
+Wire Wire Line
+	7200 1000 7200 1050
 Wire Wire Line
 	6500 2300 6550 2300
@@
 Connection ~ 4550 4250
 Wire Wire Line
-	6950 2400 7100 2400
+	7050 2300 7200 2300
 $Comp
 L Swadge_Parts:SW_DPDT_x2 SW5
@@
 Wire Notes Line
 	7950 500  6100 500
-Wire Notes Line
-	6100 500  6100 2500
-Wire Notes Line
-	6100 2500 7950 2500
-Wire Notes Line
-	7950 500  7950 2500
 Text Notes 4250 600  0    50   ~ 0
 Power Switches
@@
 Wire Wire Line
 	1200 3300 1300 3300
-$Comp
-L Swadge_Parts:SW_DPDT_x2 SW1
-U 1 1 5C519EE6
-P 6750 1000
-F 0 "SW1" H 6750 1285 50  0000 C CNN
-F 1 "SW_DPDT_x2" H 6750 1194 50  0000 C CNN
-F 2 "Swadge_Parts:JS202011CQN" H 6750 1000 50  0001 C CNN
-F 3 "https://www.ckswitches.com/media/1422/js.pdf" H 6750 1000 50  0001 C CNN
-F 4 "45" H 0   0   50  0001 C CNN "Cost100"
-F 5 "401-2001-ND" H 0   0   50  0001 C CNN "Digikey"
-F 6 "Y" H 0   0   50  0001 C CNN "Substitutable"
-	1    6750 1000
-	1    0    0    -1
-$EndComp
-$Comp
-L Swadge_Parts:SW_DPDT_x2 SW2
-U 1 1 5C519F7A
-P 6750 2300
-F 0 "SW2" H 6750 2585 50  0000 C CNN
-F 1 "SW_DPDT_x2" H 6750 2494 50  0000 C CNN
-F 2 "Swadge_Parts:JS202011CQN" H 6750 2300 50  0001 C CNN
-F 3 "https://www.ckswitches.com/media/1422/js.pdf" H 6750 2300 50  0001 C CNN
-F 4 "45" H 0   0   50  0001 C CNN "Cost100"
-F 5 "401-2001-ND" H 0   0   50  0001 C CNN "Digikey"
-F 6 "Y" H 0   0   50  0001 C CNN "Substitutable"
-	1    6750 2300
-	1    0    0    -1
-$EndComp
-$Comp
-L Swadge_Parts:SW_DPDT_x2 SW1
-U 2 1 5C51AA60
-P 7650 1650
-AR Path="/5C51A884" Ref="SW1"  Part="2"
-AR Path="/5C51AA60" Ref="SW3"  Part="2"
-F 0 "SW3" H 7650 1935 50  0000 C CNN
-F 1 "SW_DPDT_x2" H 7650 1844 50  0000 C CNN
-F 2 "Swadge_Parts:JS202011CQN" H 7650 1650 50  0001 C CNN
-F 3 "https://www.ckswitches.com/media/1422/js.pdf" H 7650 1650 50  0001 C CNN
-F 4 "45" H 0   0   50  0001 C CNN "Cost100"
-F 5 "401-2001-ND" H 0   0   50  0001 C CNN "Digikey"
-F 6 "Y" H 0   0   50  0001 C CNN "Substitutable"
-	2    7650 1650
-	1    0    0    -1
-$EndComp
-$Comp
-L Swadge_Parts:SW_DPDT_x2 SW?
-U 2 1 5C51B068
-P 7650 1000
-AR Path="/5C51A884" Ref="SW?"  Part="2"
-AR Path="/5C51B068" Ref="SW1"  Part="2"
-F 0 "SW1" H 7650 1285 50  0000 C CNN
-F 1 "SW_DPDT_x2" H 7650 1194 50  0000 C CNN
-F 2 "Swadge_Parts:JS202011CQN" H 7650 1000 50  0001 C CNN
-F 3 "https://www.ckswitches.com/media/1422/js.pdf" H 7650 1000 50  0001 C CNN
-F 4 "45" H 0   0   50  0001 C CNN "Cost100"
-F 5 "401-2001-ND" H 0   0   50  0001 C CNN "Digikey"
-F 6 "Y" H 0   0   50  0001 C CNN "Substitutable"
-	2    7650 1000
-	1    0    0    -1
-$EndComp
-$Comp
-L Swadge_Parts:SW_DPDT_x2 SW2
-U 2 1 5C51B114
-P 7650 2300
-F 0 "SW2" H 7650 2585 50  0000 C CNN
-F 1 "SW_DPDT_x2" H 7650 2494 50  0000 C CNN
-F 2 "Swadge_Parts:JS202011CQN" H 7650 2300 50  0001 C CNN
-F 3 "https://www.ckswitches.com/media/1422/js.pdf" H 7650 2300 50  0001 C CNN
-F 4 "45" H 0   0   50  0001 C CNN "Cost100"
-F 5 "401-2001-ND" H 0   0   50  0001 C CNN "Digikey"
-F 6 "Y" H 0   0   50  0001 C CNN "Substitutable"
-	2    7650 2300
-	1    0    0    -1
-$EndComp
-$Comp
-L Swadge_Parts:SW_DPDT_x2 SW?
-U 1 1 5C51B164
-P 6750 1650
-AR Path="/5C51A884" Ref="SW?"  Part="2"
-AR Path="/5C51B164" Ref="SW3"  Part="1"
-F 0 "SW3" H 6750 1935 50  0000 C CNN
-F 1 "SW_DPDT_x2" H 6750 1844 50  0000 C CNN
-F 2 "Swadge_Parts:JS202011CQN" H 6750 1650 50  0001 C CNN
-F 3 "https://www.ckswitches.com/media/1422/js.pdf" H 6750 1650 50  0001 C CNN
-F 4 "45" H 0   0   50  0001 C CNN "Cost100"
-F 5 "401-2001-ND" H 0   0   50  0001 C CNN "Digikey"
-F 6 "Y" H 0   0   50  0001 C CNN "Substitutable"
-	1    6750 1650
-	1    0    0    -1
-$EndComp
 Connection ~ 4050 4150
 Connection ~ 4050 3950
@@
 	3000 5850 3000 5950
 Connection ~ 3000 5950
-Text GLabel 7100 2400 2    50   Input ~ 0
+Text GLabel 7200 2300 2    50   Input ~ 0
 3.3V
 $Comp
@@
 Wire Notes Line
 	4500 2100 4500 1950
+$Comp
+L Swadge_Parts:4-1437565-2 SW1
+U 1 1 5CA361AC
+P 6800 1100
+F 0 "SW1" H 6800 1415 50  0000 C CNN
+F 1 "4-1437565-2" H 6800 1324 50  0000 C CNN
+F 2 "Swadge_Parts:SW_4-1437565-2" H 6800 1100 50  0001 L BNN
+F 3 "https://www.te.com/commerce/DocumentDelivery/DDEController?Action=srchrtrv&DocNm=2-1437565-7&DocType=Customer+Drawing&DocLang=English" H 6800 1100 50  0001 L BNN
+F 4 "Switch Tactile OFF _ON_ SPST Round Button Gull Wing 0.05A 24VDC 1VA 9.18N SMD T/R" H 6800 1100 50  0001 L BNN "Description"
+F 5 "TE Connectivity" H 6800 1100 50  0001 L BNN "Manufacturer"
+F 6 "FSM4JSMATR" H 6800 1100 50  0001 L BNN "MPN"
+F 7 "450-1759-1-ND" H 7440 2070 50  0001 C CNN "Digikey"
+F 8 "34" H 6800 1100 10  0001 C CNN "Cost100"
+F 9 "Y" H 6800 1100 10  0001 C CNN "Substitutable"
+	1    6800 1100
+	1    0    0    -1
+$EndComp
+$Comp
+L Swadge_Parts:4-1437565-2 SW2
+U 1 1 5CA3636E
+P 6800 1750
+F 0 "SW2" H 6800 2065 50  0000 C CNN
+F 1 "4-1437565-2" H 6800 1974 50  0000 C CNN
+F 2 "Swadge_Parts:SW_4-1437565-2" H 6800 1750 50  0001 L BNN
+F 3 "https://www.te.com/commerce/DocumentDelivery/DDEController?Action=srchrtrv&DocNm=2-1437565-7&DocType=Customer+Drawing&DocLang=English" H 6800 1750 50  0001 L BNN
+F 4 "Switch Tactile OFF _ON_ SPST Round Button Gull Wing 0.05A 24VDC 1VA 9.18N SMD T/R" H 6800 1750 50  0001 L BNN "Description"
+F 5 "TE Connectivity" H 6800 1750 50  0001 L BNN "Manufacturer"
+F 6 "FSM4JSMATR" H 6800 1750 50  0001 L BNN "MPN"
+F 7 "450-1759-1-ND" H 7440 2720 50  0001 C CNN "Digikey"
+F 8 "34" H 6800 1750 10  0001 C CNN "Cost100"
+F 9 "Y" H 6800 1750 10  0001 C CNN "Substitutable"
+	1    6800 1750
+	1    0    0    -1
+$EndComp
+$Comp
+L Swadge_Parts:4-1437565-2 SW3
+U 1 1 5CA363D2
+P 6800 2400
+F 0 "SW3" H 6800 2715 50  0000 C CNN
+F 1 "4-1437565-2" H 6800 2624 50  0000 C CNN
+F 2 "Swadge_Parts:SW_4-1437565-2" H 6800 2400 50  0001 L BNN
+F 3 "https://www.te.com/commerce/DocumentDelivery/DDEController?Action=srchrtrv&DocNm=2-1437565-7&DocType=Customer+Drawing&DocLang=English" H 6800 2400 50  0001 L BNN
+F 4 "Switch Tactile OFF _ON_ SPST Round Button Gull Wing 0.05A 24VDC 1VA 9.18N SMD T/R" H 6800 2400 50  0001 L BNN "Description"
+F 5 "TE Connectivity" H 6800 2400 50  0001 L BNN "Manufacturer"
+F 6 "FSM4JSMATR" H 6800 2400 50  0001 L BNN "MPN"
+F 7 "450-1759-1-ND" H 7440 3370 50  0001 C CNN "Digikey"
+F 8 "34" H 6800 2400 10  0001 C CNN "Cost100"
+F 9 "Y" H 6800 2400 10  0001 C CNN "Substitutable"
+	1    6800 2400
+	1    0    0    -1
+$EndComp
+Wire Wire Line
+	7050 2300 7050 2500
+Connection ~ 7050 2300
+Wire Wire Line
+	6550 2500 6550 2300
+Connection ~ 6550 2300
+Wire Wire Line
+	6550 1850 6550 1650
+Connection ~ 6550 1650
+Wire Wire Line
+	7050 1650 7050 1850
+Connection ~ 7050 1650
+Wire Wire Line
+	7050 1200 7050 1000
+Connection ~ 7050 1000
+Wire Wire Line
+	6550 1000 6550 1200
+Connection ~ 6550 1000
+Wire Notes Line
+	6100 500  6100 2600
+Wire Notes Line
+	7500 500  7500 2600
+Wire Notes Line
+	7500 2600 6100 2600
 $EndSCHEMATC
