File: hardware/swadge-programmer.sch (KiCad schematic (older format))
At the start: 24 parts, among them J1 USB_B_Micro, J2 Conn_02x21_Top_Bottom, J3 Conn_02x21_Top_Bottom, SW1 4-1437565-2, SW2 4-1437565-2, SW3 4-1437565-2, SW4 SW_DPDT_x2, SW5 SW_DPDT_x2, U1 BUS_PCIexpress, U2 CP2102N-A01-GQFN24

Commit message: #5 Added FTDI-ordered breakout of all UART pins
Parts:
- added J4: ftdi-header, Swadge_Parts:ftdi-header, symbol Swadge_Parts:ftdi-header
Connections:
- net labels added: CTS, RTS
- wire segments 178 -> 186
Changed lines of the file:
@@
 Wire Notes Line
 	7500 2600 6100 2600
+$Comp
+L Swadge_Parts:ftdi-header J4
+U 1 1 5CAF207F
+P 1750 1050
+F 0 "J4" H 1794 635 50  0000 C CNN
+F 1 "ftdi-header" H 1794 726 50  0000 C CNN
+F 2 "Swadge_Parts:ftdi-header" H 1700 1750 50  0001 C CNN
+F 3 "https://www.ftdichip.com/Support/Documents/DataSheets/Cables/DS_TTL-232R_CABLES.pdf" H 1600 1650 50  0001 C CNN
+F 4 "n/a" H 1950 1550 50  0001 C CNN "Digikey"
+F 5 "0" H 2050 1650 50  0001 C CNN "Cost100"
+F 6 "n" H 2150 1750 50  0001 C CNN "Substitutable"
+F 7 "y" H 2250 1850 50  0001 C CNN "NOBOM"
+	1    1750 1050
+	-1   0    0    1
+$EndComp
+Text GLabel 1900 1050 2    50   Input ~ 0
+TX
+Text GLabel 1900 950  2    50   Input ~ 0
+RX
+Wire Wire Line
+	1850 950  1900 950
+Wire Wire Line
+	1850 1050 1900 1050
+$Comp
+L power:GND #PWR0101
+U 1 1 5CB0C37E
+P 1900 1350
+F 0 "#PWR0101" H 1900 1100 50  0001 C CNN
+F 1 "GND" H 1905 1177 50  0000 C CNN
+F 2 "" H 1900 1350 50  0001 C CNN
+F 3 "" H 1900 1350 50  0001 C CNN
+	1    1900 1350
+	1    0    0    -1
+$EndComp
+Wire Wire Line
+	1850 1350 1900 1350
+Text GLabel 3800 1850 2    50   Input ~ 0
+RTS
+Text GLabel 3800 1750 2    50   Input ~ 0
+CTS
+Wire Wire Line
+	3800 1750 3750 1750
+Wire Wire Line
+	3800 1850 3750 1850
+Text GLabel 1900 1250 2    50   Input ~ 0
+CTS
+Text GLabel 1900 850  2    50   Input ~ 0
+RTS
+Wire Wire Line
+	1850 850  1900 850
+Wire Wire Line
+	1850 1250 1900 1250
+$Comp
+L power:+5V #PWR0102
+U 1 1 5CB4B3FE
+P 2150 1150
+F 0 "#PWR0102" H 2150 1000 50  0001 C CNN
+F 1 "+5V" H 2165 1323 50  0000 C CNN
+F 2 "" H 2150 1150 50  0001 C CNN
+F 3 "" H 2150 1150 50  0001 C CNN
+	1    2150 1150
+	1    0    0    -1
+$EndComp
+Wire Wire Line
+	1850 1150 2150 1150
 $EndSCHEMATC

Commit message: #1 #2 #3 #5 #6 #7 #16 Routed PCB
Changed lines of the file:
@@
 	3000 5850 3000 5950
 Connection ~ 3000 5950
-Text GLabel 7200 2300 2    50   Input ~ 0
-3.3V
 $Comp
 L Swadge_Parts:R_US R4
@@
 Wire Wire Line
 	1850 1150 2150 1150
+$Comp
+L power:+3.3V #PWR?
+U 1 1 5CB557DC
+P 7200 2300
+F 0 "#PWR?" H 7200 2150 50  0001 C CNN
+F 1 "+3.3V" H 7215 2473 50  0000 C CNN
+F 2 "" H 7200 2300 50  0001 C CNN
+F 3 "" H 7200 2300 50  0001 C CNN
+	1    7200 2300
+	1    0    0    -1
+$EndComp
 $EndSCHEMATC
