File: hardware/swadge-programmer.sch (KiCad schematic (older format))
At the start: 25 parts, among them J1 USB_B_Micro, J2 Conn_02x21_Top_Bottom, J3 Conn_02x21_Top_Bottom, J4 ftdi-header, SW1 4-1437565-2, SW2 4-1437565-2, SW3 4-1437565-2, SW4 SW_DPDT_x2, SW5 SW_DPDT_x2, U2 CP2102N-A01-GQFN24

Commit message: Swapped RX/TX on FTDI header, added voltage jumper selector
Parts:
- added J5: Conn_01x03_Male, Swadge_Parts:PinHeader_1x03_P2.54mm_Vertical, symbol Swadge_Parts:Conn_01x03_Male
- renumbered U to U1
Connections:
- wire segments 186 -> 191
Other:
- note added: "UART data lines are\nlabeled from the\nperspective of the devkit"
Changed lines of the file:
@@
 EESchema Schematic File Version 4
+LIBS:swadge-programmer-cache
 EELAYER 26 0
 EELAYER END
@@
 $EndComp
 $Comp
-L Swadge_Parts:BUS_PCIexpress U
+L Swadge_Parts:BUS_PCIexpress U1
 U 1 1 5C4297AA
 P 1200 4950
-F 0 "U" H 1200 6025 50  0000 C CNN
+F 0 "U1" H 1200 6025 50  0000 C CNN
 F 1 "BUS_PCIexpress" H 1200 5934 50  0000 C CNN
 F 2 "Swadge_Parts:BUS_PCIexpress" H 1200 5300 50  0001 C CNN
@@
 L power:+5V #PWR09
 U 1 1 5C469190
-P 1300 1650
-F 0 "#PWR09" H 1300 1500 50  0001 C CNN
-F 1 "+5V" H 1315 1823 50  0000 C CNN
-F 2 "" H 1300 1650 50  0001 C CNN
-F 3 "" H 1300 1650 50  0001 C CNN
-	1    1300 1650
+P 1550 1500
+F 0 "#PWR09" H 1550 1350 50  0001 C CNN
+F 1 "+5V" H 1565 1673 50  0000 C CNN
+F 2 "" H 1550 1500 50  0001 C CNN
+F 3 "" H 1550 1500 50  0001 C CNN
+	1    1550 1500
 	1    0    0    -1
 $EndComp
@@
 L Swadge_Parts:ftdi-header J4
 U 1 1 5CAF207F
-P 1750 1050
-F 0 "J4" H 1794 635 50  0000 C CNN
-F 1 "ftdi-header" H 1794 726 50  0000 C CNN
-F 2 "Swadge_Parts:ftdi-header" H 1700 1750 50  0001 C CNN
-F 3 "https://www.ftdichip.com/Support/Documents/DataSheets/Cables/DS_TTL-232R_CABLES.pdf" H 1600 1650 50  0001 C CNN
-F 4 "n/a" H 1950 1550 50  0001 C CNN "Digikey"
-F 5 "0" H 2050 1650 50  0001 C CNN "Cost100"
-F 6 "n" H 2150 1750 50  0001 C CNN "Substitutable"
-F 7 "y" H 2250 1850 50  0001 C CNN "NOBOM"
-	1    1750 1050
+P 850 1150
+F 0 "J4" H 894 735 50  0000 C CNN
+F 1 "ftdi-header" H 894 826 50  0000 C CNN
+F 2 "Swadge_Parts:ftdi-header" H 800 1850 50  0001 C CNN
+F 3 "https://www.ftdichip.com/Support/Documents/DataSheets/Cables/DS_TTL-232R_CABLES.pdf" H 700 1750 50  0001 C CNN
+F 4 "n/a" H 1050 1650 50  0001 C CNN "Digikey"
+F 5 "0" H 1150 1750 50  0001 C CNN "Cost100"
+F 6 "n" H 1250 1850 50  0001 C CNN "Substitutable"
+F 7 "y" H 1350 1950 50  0001 C CNN "NOBOM"
+	1    850  1150
 	-1   0    0    1
 $EndComp
-Text GLabel 1900 1050 2    50   Input ~ 0
+Text GLabel 1000 1050 2    50   Input ~ 0
 TX
-Text GLabel 1900 950  2    50   Input ~ 0
+Text GLabel 1000 1150 2    50   Input ~ 0
 RX
 Wire Wire Line
-	1850 950  1900 950
-Wire Wire Line
-	1850 1050 1900 1050
+	950  1050 1000 1050
+Wire Wire Line
+	950  1150 1000 1150
 $Comp
 L power:GND #PWR0101
 U 1 1 5CB0C37E
-P 1900 1350
-F 0 "#PWR0101" H 1900 1100 50  0001 C CNN
-F 1 "GND" H 1905 1177 50  0000 C CNN
-F 2 "" H 1900 1350 50  0001 C CNN
-F 3 "" H 1900 1350 50  0001 C CNN
-	1    1900 1350
-	1    0    0    -1
-$EndComp
-Wire Wire Line
-	1850 1350 1900 1350
+P 1000 1450
+F 0 "#PWR0101" H 1000 1200 50  0001 C CNN
+F 1 "GND" H 1005 1277 50  0000 C CNN
+F 2 "" H 1000 1450 50  0001 C CNN
+F 3 "" H 1000 1450 50  0001 C CNN
+	1    1000 1450
+	1    0    0    -1
+$EndComp
+Wire Wire Line
+	950  1450 1000 1450
+Text GLabel 3800 1750 2    50   Input ~ 0
+RTS
 Text GLabel 3800 1850 2    50   Input ~ 0
+CTS
+Wire Wire Line
+	3800 1750 3750 1750
+Wire Wire Line
+	3800 1850 3750 1850
+Text GLabel 1000 950  2    50   Input ~ 0
+CTS
+Text GLabel 1000 1350 2    50   Input ~ 0
 RTS
-Text GLabel 3800 1750 2    50   Input ~ 0
-CTS
-Wire Wire Line
-	3800 1750 3750 1750
-Wire Wire Line
-	3800 1850 3750 1850
-Text GLabel 1900 1250 2    50   Input ~ 0
-CTS
-Text GLabel 1900 850  2    50   Input ~ 0
-RTS
-Wire Wire Line
-	1850 850  1900 850
-Wire Wire Line
-	1850 1250 1900 1250
-$Comp
-L power:+5V #PWR0102
-U 1 1 5CB4B3FE
-P 2150 1150
-F 0 "#PWR0102" H 2150 1000 50  0001 C CNN
-F 1 "+5V" H 2165 1323 50  0000 C CNN
-F 2 "" H 2150 1150 50  0001 C CNN
-F 3 "" H 2150 1150 50  0001 C CNN
-	1    2150 1150
-	1    0    0    -1
-$EndComp
-Wire Wire Line
-	1850 1150 2150 1150
-$Comp
-L power:+3.3V #PWR?
+Wire Wire Line
+	950  950  1000 950
+Wire Wire Line
+	950  1350 1000 1350
+$Comp
+L power:+3.3V #PWR0102
 U 1 1 5CB557DC
 P 7200 2300
-F 0 "#PWR?" H 7200 2150 50  0001 C CNN
+F 0 "#PWR0102" H 7200 2150 50  0001 C CNN
 F 1 "+3.3V" H 7215 2473 50  0000 C CNN
 F 2 "" H 7200 2300 50  0001 C CNN
@@
 	1    0    0    -1
 $EndComp
+Text Notes 1650 850  0    50   ~ 0
+UART data lines are\nlabeled from the\nperspective of the devkit
+$Comp
+L Swadge_Parts:Conn_01x03_Male J5
+U 1 1 5CA515AE
+P 2000 1350
+F 0 "J5" H 1973 1280 50  0000 R CNN
+F 1 "Conn_01x03_Male" H 2200 1100 50  0000 R CNN
+F 2 "Swadge_Parts:PinHeader_1x03_P2.54mm_Vertical" H 1900 1450 50  0001 C CNN
+F 3 "https://www.metz-connect.com/us/system/files/productfiles/Data_sheet_PR202XXVBNN_PR202XXVBNN_OFF-024022P.pdf" H 2000 1550 50  0001 C CNN
+F 4 "1849-1003-ND" H 2100 1650 50  0001 C CNN "Digikey"
+F 5 "10" H 2200 1750 50  0001 C CNN "Cost100"
+F 6 "Y" H 2300 1850 50  0001 C CNN "Substitutable"
+	1    2000 1350
+	-1   0    0    1
+$EndComp
+Wire Wire Line
+	1750 1650 1750 1450
+Wire Wire Line
+	950  1250 1800 1250
+Wire Wire Line
+	1800 1450 1750 1450
+Wire Wire Line
+	1800 1350 1700 1350
+Wire Wire Line
+	1700 1350 1700 1500
+Wire Wire Line
+	1700 1500 1550 1500
 $EndSCHEMATC

Commit message: #17 Reordered PCIe connector on programmer
Parts:
- removed J2, J3: Conn_02x21_Top_Bottom, Swadge_Parts:PinHeader_2x21_P2.54mm_Vertical, symbol Swadge_Parts:Conn_02x21_Top_Bottom
- added J2, J3: Conn_02x15_Top_Bottom, Swadge_Parts:PinHeader_2x15_P2.54mm_Vertical, symbol Swadge_Parts:Conn_02x15_Top_Bottom
- U1: footprint Swadge_Parts:BUS_PCIexpress -> Swadge_Parts:10018784-10210TLF
Connections:
- net labels added: _RES
- net labels removed: CS0, GPIO0, GPIO15, GPIO2, MISO, MOSI, SCLK
- wire segments 191 -> 173
- no-connect marks 16 -> 10
Other:
- moved on the sheet: R4, R5

Commit message: #4 Add Rubber foot to hole part, update digikey values
Parts:
- H1, H2, H3, H4: Cost100 0 -> 9; Digikey n/a -> 2042-1007-ND; NOBOM y -> (none)
Changed lines of the file:
@@
 EESchema Schematic File Version 4
+LIBS:swadge-programmer-cache
 EELAYER 29 0
 EELAYER END
@@
 F 1 "USB_B_Micro" H 855 3026 50  0000 C CNN
 F 2 "Swadge_Parts:USB_Micro-B_Molex_47346-0001" H 950 2600 50  0001 C CNN
-F 3 "https://www.molex.com/pdm_docs/sd/473460001_sd.pdf" H 950 2600 50  0001 C CNN
+F 3 "https://www.digikey.com/product-detail/en/molex-llc/0473460001/WM17141CT-ND/1782474" H 950 2600 50  0001 C CNN
 F 4 "112" H 0   0   50  0001 C CNN "Cost100"
 F 5 "WM17141CT-ND" H 0   0   50  0001 C CNN "Digikey"
@@
 F 1 "SP0503BAHT" H 1505 3055 50  0000 L CNN
 F 2 "Swadge_Parts:SOT-143" H 1525 3050 50  0001 L CNN
-F 3 "https://www.littelfuse.com/~/media/files/littelfuse/technical%20resources/documents/data%20sheets/sp05xxba.pdf" H 1425 3225 50  0001 C CNN
+F 3 "http://www.littelfuse.com/~/media/files/littelfuse/technical%20resources/documents/data%20sheets/sp05xxba.pdf" H 1425 3225 50  0001 C CNN
 F 4 "95" H 0   0   50  0001 C CNN "Cost100"
 F 5 "F2715CT-ND" H 0   0   50  0001 C CNN "Digikey"
@@
 F 1 "22.1k" H 1368 1755 50  0000 L CNN
 F 2 "Swadge_Parts:R_0603_1608Metric" V 1340 1790 50  0001 C CNN
-F 3 "" H 1300 1800 50  0001 C CNN
+F 3 "~" H 1300 1800 50  0001 C CNN
 F 4 "10" H 0   0   50  0001 C CNN "Cost100"
 F 5 "RMCF0603FT22K1CT-ND" H 0   0   50  0001 C CNN "Digikey"
@@
 F 1 "47.5k" H 1368 2155 50  0000 L CNN
 F 2 "Swadge_Parts:R_0603_1608Metric" V 1340 2190 50  0001 C CNN
-F 3 "" H 1300 2200 50  0001 C CNN
+F 3 "~" H 1300 2200 50  0001 C CNN
 F 4 "10" H 0   0   50  0001 C CNN "Cost100"
 F 5 "P47.5KHCT-ND" H 0   0   50  0001 C CNN "Digikey"
@@
 F 1 "CP2102N-A01-GQFN24" H 3650 3050 50  0000 C CNN
 F 2 "Swadge_Parts:QFN-24-1EP_4x4mm_P0.5mm_EP2.6x2.6mm" H 3600 1450 50  0001 L CNN
-F 3 "https://www.silabs.com/documents/public/data-sheets/cp2102n-datasheet.pdf" H 3200 1200 50  0001 C CNN
+F 3 "http://www.silabs.com/support%20documents/technicaldocs/cp2102n-datasheet.pdf" H 3200 1200 50  0001 C CNN
 F 4 "135" H 0   0   50  0001 C CNN "Cost100"
 F 5 "336-4737-1-ND" H 0   0   50  0001 C CNN "Digikey"
@@
 F 1 "1k" H 2482 1295 50  0000 R CNN
 F 2 "Swadge_Parts:R_0603_1608Metric" V 2590 1240 50  0001 C CNN
-F 3 "" H 2550 1250 50  0001 C CNN
+F 3 "~" H 2550 1250 50  0001 C CNN
 F 4 "10" H 0   0   50  0001 C CNN "Cost100"
 F 5 "311-1.00KHRCT-ND" H 0   0   50  0001 C CNN "Digikey"
@@
 F 1 "4.7u" H 2265 1755 50  0000 L CNN
 F 2 "Swadge_Parts:C_0603_1608Metric" H 2188 1650 50  0001 C CNN
-F 3 "" H 2150 1800 50  0001 C CNN
+F 3 "~" H 2150 1800 50  0001 C CNN
 F 4 "10" H 0   0   50  0001 C CNN "Cost100"
 F 5 "1276-1045-1-ND" H 0   0   50  0001 C CNN "Digikey"
@@
 F 1 "0.1u" H 1865 1755 50  0000 L CNN
 F 2 "Swadge_Parts:C_0603_1608Metric" H 1788 1650 50  0001 C CNN
-F 3 "" H 1750 1800 50  0001 C CNN
+F 3 "~" H 1750 1800 50  0001 C CNN
 F 4 "10" H 0   0   50  0001 C CNN "Cost100"
 F 5 "1276-1000-1-ND" H 0   0   50  0001 C CNN "Digikey"
@@
 F 1 "4.7u" H 3865 955 50  0000 L CNN
 F 2 "Swadge_Parts:C_0603_1608Metric" H 3788 850 50  0001 C CNN
-F 3 "" H 3750 1000 50  0001 C CNN
+F 3 "~" H 3750 1000 50  0001 C CNN
 F 4 "10" H 0   0   50  0001 C CNN "Cost100"
 F 5 "1276-1045-1-ND" H 0   0   50  0001 C CNN "Digikey"
@@
 F 1 "0.1u" H 3415 955 50  0000 L CNN
 F 2 "Swadge_Parts:C_0603_1608Metric" H 3338 850 50  0001 C CNN
-F 3 "" H 3300 1000 50  0001 C CNN
+F 3 "~" H 3300 1000 50  0001 C CNN
 F 4 "10" H 0   0   50  0001 C CNN "Cost100"
 F 5 "1276-1000-1-ND" H 0   0   50  0001 C CNN "Digikey"
@@
 F 1 "1" V 1500 4800 50  0000 L CNN
 F 2 "Swadge_Parts:R_Axial_DIN0207_L6.3mm_D2.5mm_P10.16mm_Horizontal" V 1640 4890 50  0001 C CNN
-F 3 "" H 1600 4900 50  0001 C CNN
+F 3 "~" H 1600 4900 50  0001 C CNN
 F 4 "10" H 0   800 50  0001 C CNN "Cost100"
 F 5 "RNF14FTD1R00CT-ND" H 0   800 50  0001 C CNN "Digikey"
@@
 F 1 "1" V 1550 5800 50  0000 L CNN
 F 2 "Swadge_Parts:R_Axial_DIN0207_L6.3mm_D2.5mm_P10.16mm_Horizontal" V 1690 5890 50  0001 C CNN
-F 3 "" H 1650 5900 50  0001 C CNN
+F 3 "~" H 1650 5900 50  0001 C CNN
 F 4 "10" H 50  700 50  0001 C CNN "Cost100"
 F 5 "RNF14FTD1R00CT-ND" H 50  700 50  0001 C CNN "Digikey"
@@
 F 1 "Hole" H 4990 2555 50  0000 L CNN
 F 2 "Swadge_Parts:Hole" H 4850 2600 50  0001 C CNN
-F 3 "" H 4850 2600 50  0001 C CNN
-F 4 "0" H 0   0   50  0001 C CNN "Cost100"
-F 5 "n/a" H 0   0   50  0001 C CNN "Digikey"
-F 6 "y" H 0   0   50  0001 C CNN "NOBOM"
-F 7 "Y" H 0   0   50  0001 C CNN "Substitutable"
+F 3 "https://www.bumperspecialties.com/wp-content/uploads/2017/01/Bumper-Technical-Drawing-BS02.pdf" H 4850 2600 50  0001 C CNN
+F 4 "9" H 0   0   50  0001 C CNN "Cost100"
+F 5 "2042-1007-ND" H 0   0   50  0001 C CNN "Digikey"
+F 6 "Y" H 0   0   50  0001 C CNN "Substitutable"
 	1    4850 2600
 	1    0    0    -1
@@
 F 1 "Hole" H 5490 2555 50  0000 L CNN
 F 2 "Swadge_Parts:Hole" H 5350 2600 50  0001 C CNN
-F 3 "" H 5350 2600 50  0001 C CNN
-F 4 "0" H 0   0   50  0001 C CNN "Cost100"
-F 5 "n/a" H 0   0   50  0001 C CNN "Digikey"
-F 6 "y" H 0   0   50  0001 C CNN "NOBOM"
-F 7 "Y" H 0   0   50  0001 C CNN "Substitutable"
+F 3 "https://www.bumperspecialties.com/wp-content/uploads/2017/01/Bumper-Technical-Drawing-BS02.pdf" H 5350 2600 50  0001 C CNN
+F 4 "9" H 0   0   50  0001 C CNN "Cost100"
+F 5 "2042-1007-ND" H 0   0   50  0001 C CNN "Digikey"
+F 6 "Y" H 0   0   50  0001 C CNN "Substitutable"
 	1    5350 2600
 	1    0    0    -1
@@
 F 1 "Hole" H 4990 2855 50  0000 L CNN
 F 2 "Swadge_Parts:Hole" H 4850 2900 50  0001 C CNN
-F 3 "" H 4850 2900 50  0001 C CNN
-F 4 "0" H 0   0   50  0001 C CNN "Cost100"
-F 5 "n/a" H 0   0   50  0001 C CNN "Digikey"
-F 6 "y" H 0   0   50  0001 C CNN "NOBOM"
-F 7 "Y" H 0   0   50  0001 C CNN "Substitutable"
+F 3 "https://www.bumperspecialties.com/wp-content/uploads/2017/01/Bumper-Technical-Drawing-BS02.pdf" H 4850 2900 50  0001 C CNN
+F 4 "9" H 0   0   50  0001 C CNN "Cost100"
+F 5 "2042-1007-ND" H 0   0   50  0001 C CNN "Digikey"
+F 6 "Y" H 0   0   50  0001 C CNN "Substitutable"
 	1    4850 2900
 	1    0    0    -1
@@
 F 1 "Hole" H 5490 2855 50  0000 L CNN
 F 2 "Swadge_Parts:Hole" H 5350 2900 50  0001 C CNN
-F 3 "" H 5350 2900 50  0001 C CNN
-F 4 "0" H 0   0   50  0001 C CNN "Cost100"
-F 5 "n/a" H 0   0   50  0001 C CNN "Digikey"
-F 6 "y" H 0   0   50  0001 C CNN "NOBOM"
-F 7 "Y" H 0   0   50  0001 C CNN "Substitutable"
+F 3 "https://www.bumperspecialties.com/wp-content/uploads/2017/01/Bumper-Technical-Drawing-BS02.pdf" H 5350 2900 50  0001 C CNN
+F 4 "9" H 0   0   50  0001 C CNN "Cost100"
+F 5 "2042-1007-ND" H 0   0   50  0001 C CNN "Digikey"
+F 6 "Y" H 0   0   50  0001 C CNN "Substitutable"
 	1    5350 2900
 	1    0    0    -1
@@
 F 1 "4-1437565-2" H 6800 1324 50  0000 C CNN
 F 2 "Swadge_Parts:SW_4-1437565-2" H 6800 1100 50  0001 L BNN
-F 3 "https://www.te.com/commerce/DocumentDelivery/DDEController?Action=srchrtrv&DocNm=2-1437565-7&DocType=Customer+Drawing&DocLang=English" H 6800 1100 50  0001 L BNN
+F 3 "https://www.diodes.com/assets/Datasheets/AP2114.pdf" H 6800 1100 50  0001 L BNN
 F 4 "Switch Tactile OFF _ON_ SPST Round Button Gull Wing 0.05A 24VDC 1VA 9.18N SMD T/R" H 6800 1100 50  0001 L BNN "Description"
 F 5 "TE Connectivity" H 6800 1100 50  0001 L BNN "Manufacturer"
@@
 F 1 "4-1437565-2" H 6800 1974 50  0000 C CNN
 F 2 "Swadge_Parts:SW_4-1437565-2" H 6800 1750 50  0001 L BNN
-F 3 "https://www.te.com/commerce/DocumentDelivery/DDEController?Action=srchrtrv&DocNm=2-1437565-7&DocType=Customer+Drawing&DocLang=English" H 6800 1750 50  0001 L BNN
+F 3 "https://www.diodes.com/assets/Datasheets/AP2114.pdf" H 6800 1750 50  0001 L BNN
 F 4 "Switch Tactile OFF _ON_ SPST Round Button Gull Wing 0.05A 24VDC 1VA 9.18N SMD T/R" H 6800 1750 50  0001 L BNN "Description"
 F 5 "TE Connectivity" H 6800 1750 50  0001 L BNN "Manufacturer"
@@
 F 1 "4-1437565-2" H 6800 2624 50  0000 C CNN
 F 2 "Swadge_Parts:SW_4-1437565-2" H 6800 2400 50  0001 L BNN
-F 3 "https://www.te.com/commerce/DocumentDelivery/DDEController?Action=srchrtrv&DocNm=2-1437565-7&DocType=Customer+Drawing&DocLang=English" H 6800 2400 50  0001 L BNN
+F 3 "https://www.diodes.com/assets/Datasheets/AP2114.pdf" H 6800 2400 50  0001 L BNN
 F 4 "Switch Tactile OFF _ON_ SPST Round Button Gull Wing 0.05A 24VDC 1VA 9.18N SMD T/R" H 6800 2400 50  0001 L BNN "Description"
 F 5 "TE Connectivity" H 6800 2400 50  0001 L BNN "Manufacturer"
@@
 F 1 "Conn_01x03_Male" H 2200 1100 50  0000 R CNN
 F 2 "Swadge_Parts:PinHeader_1x03_P2.54mm_Vertical" H 1900 1450 50  0001 C CNN
-F 3 "https://www.metz-connect.com/us/system/files/productfiles/Data_sheet_PR202XXVBNN_PR202XXVBNN_OFF-024022P.pdf" H 2000 1550 50  0001 C CNN
+F 3 "~" H 2000 1550 50  0001 C CNN
 F 4 "1849-1003-ND" H 2100 1650 50  0001 C CNN "Digikey"
 F 5 "10" H 2200 1750 50  0001 C CNN "Cost100"
