File: hardware/swadge-screen-test.kicad_pcb (KiCad board)
At the start: 2 copper layers, 56.8 x 49.2 mm, 12 parts, among them U2 DISP_OLED_UG-2864HSWEG01

Commit message: Added backside of screen-test board
Parts:
- added REF**: R_0603_1608Metric, Resistor_SMD:R_0603_1608Metric, B.Cu at (203.2, 70.6)
- added REF**: R_0603_1608Metric, Resistor_SMD:R_0603_1608Metric, B.Cu at (205.0, 69.8)
- added REF**: R_0603_1608Metric, Resistor_SMD:R_0603_1608Metric, B.Cu at (219.2, 69.8)
- added REF**: R_0603_1608Metric, Resistor_SMD:R_0603_1608Metric, B.Cu at (221.0, 69.0)
- added REF**: C_0805_2012Metric, Capacitor_SMD:C_0805_2012Metric, B.Cu at (226.5, 71.6)
- added REF**: C_0805_2012Metric, Capacitor_SMD:C_0805_2012Metric, B.Cu at (223.8, 68.8)
- added REF**: C_0805_2012Metric, Capacitor_SMD:C_0805_2012Metric, B.Cu at (197.7, 71.6)
- added REF**: C_0805_2012Metric, Capacitor_SMD:C_0805_2012Metric, B.Cu at (200.4, 68.8)
- added U2: DISP_OLED_UG-2864HSWEG01, Swadge_Parts:oled-flat, B.Cu at (212.1, 69.8)
Routing:
- added copper zone on B.Cu, net GND
