File: hardware/swadge-banana/swadge-banana.sch (KiCad schematic (older format))
At the start: 42 parts, among them J1 USB_B_Micro, SW1 4-1437565-2, SW2 4-1437565-2, SW3 4-1437565-2, SW4 SW_SPDT, U1 ESP-13-WROOM-02D, U2 DISP_OLED_UG-2864HSWEG01, U3 BUS_PCIexpress, U4 QMA6981, U5 AP1117-33

Commit message: Reset banana board to a blank slate for cnlohr
Parts:
- removed SW1, SW3: 4-1437565-2, Swadge_Parts:SW_4-1437565-2, symbol Swadge_Parts:4-1437565-2
- added H1: Headband, Swadge_Parts:Headband, symbol Swadge_Parts:Headband
- added LS1: Speaker, Swadge_Parts:Buzzer_12x9.5RM7.6, symbol Swadge_Parts:Speaker
- added Q1: Q_NPN_BEC, Swadge_Parts:SOT-23, symbol Swadge_Parts:Q_NPN_BEC
- added R7: 100, Swadge_Parts:R_0603_1608Metric, symbol Swadge_Parts:R_US
- added S2, S3: B3FS-4002P, Swadge_Parts:B3FS4002P, symbol Swadge_Parts:B3FS-4002P
- added U2: OLED_DISPLAY, Swadge_Parts:NULL, symbol Swadge_Parts:OLED_DISPLAY
- BT1, BT2: Notes (none) -> Use through-hole AA Battery Holder in Style of Keystone 2460
- C1, C10, C11, C12, C13, C14, C15, C16, C17, C2, C3, C7, C8, R1, R2, R3, R4, R5, R6: Notes (none) -> 0603 Package
- C18: Digikey 1276-1000-1-ND -> 1276-1085-1-ND; Notes (none) -> 0603 Package
- C4, C5, C6, C9: footprint Swadge_Parts:C_0805_2012Metric -> Swadge_Parts:C_0603_1608Metric; Notes (none) -> 0603 Package
- D1, D2, D3, D4, D5, D6: Notes Digikey item is x10 -> Use WS2812B LED. Digikey item is x10
- J1: Notes (none) -> Must use micro USB SMT-only Header
- S1: renamed from SW2; MPN FSM4JSMATR -> (none); Manufacturer TE Connectivity -> (none); Notes (none) -> Use standard SMT box tactile buttons. Similar to PTS645SM43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
- SW1: renamed from SW4; Notes (none) -> Use SPDT slide switch. Similar to PCM12SMTR
- U1: Notes (none) -> Use ESP-WROOM-02D
- U4: Notes (none) -> Use https://lcsc.com/product-detail/Others_QST-QMA6981_C310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
- U5: Notes (none) -> Use any 1117 3.3V SOT-223 regulator. I.e. AZ1117 or AP1117
- U6: renamed from U2; value DISP_OLED_UG-2864HSWEG01 -> OLED_CONNECTOR; footprint Swadge_Parts:oled-flat -> Swadge_Parts:ER-OLED0.96-1.3; symbol Swadge_Parts:DISP_OLED_UG-2864HSWEG01 -> Swadge_Parts:OLED_CONNECTOR; Adafruit https://cdn-shop.adafruit.com/datasheets/UG-2864HSWEG01.pdf -> (none); Cost100 988 -> 119; Digikey 541-3486-ND -> LCSC #C11095; Notes (none) -> Must have top contacts. same as the OLED
Connections:
- net labels added: BZR, LED_OUT, SW1
- net labels removed: SW4, SW5
- wire segments 203 -> 211
- no-connect marks 14 -> 12
Other:
- note added: "Buzzer"
- note added: "Left"
- note added: "Menu"
- note added: "Right"
- moved on the sheet: C16, C17, C18, S1, U3, U4
