File: hardware/swadge-banana/swadge-banana.sch (KiCad schematic (older format))
At the start: 46 parts, among them J1 USB_B_Micro, SW1 SW_SPDT, U1 ESP-13-WROOM-02D, U2 OLED_DISPLAY, U3 BUS_PCIexpress, U4 QMA6981, U5 AP1117-33, U6 OLED_CONNECTOR

Commit message: bump swadge-banana
Parts:
- removed C11, C13, C15: 1u, Swadge_Parts:C_0603_1608Metric, symbol Swadge_Parts:C
Connections:
- net +3V3: no longer C17.1, C18.1, C2.2, C3.2, R1.1, U1.1 (VCC), U4.7 (VDD)
- new net: C2.2, C3.2, R1.1, U1.1 (VCC)
- new net: C17.1, C18.1, U4.7 (VDD)
Changed lines of the file:
@@
 EESchema Schematic File Version 4
-LIBS:swadge-banana-cache
-EELAYER 29 0
+EELAYER 30 0
 EELAYER END
 $Descr A4 11693 8268
@@
 Wire Wire Line
 	4300 1350 4300 900
-Connection ~ 4300 900
 $Comp
 L power:GND #PWR014
@@
 $EndComp
 $Comp
-L Swadge_Parts:C C11
-U 1 1 5C3A88B1
-P 5100 1050
-F 0 "C11" H 5215 1096 50  0000 L CNN
-F 1 "1u" H 5215 1005 50  0000 L CNN
-F 2 "Swadge_Parts:C_0603_1608Metric" H 5138 900 50  0001 C CNN
-F 3 "" H 5100 1050 50  0001 C CNN
-F 4 "10" H 0   0   50  0001 C CNN "Cost100"
-F 5 "1276-1036-1-ND" H 0   0   50  0001 C CNN "Digikey"
-F 6 "Y" H 0   0   50  0001 C CNN "Substitutable"
-F 7 "0603 Package" H 5100 1050 50  0001 C CNN "Notes"
-	1    5100 1050
-	1    0    0    -1
-$EndComp
-$Comp
 L power:GND #PWR020
 U 1 1 5C3A88B7
@@
 $EndComp
 $Comp
-L Swadge_Parts:C C13
-U 1 1 5C3A9206
-P 6400 1050
-F 0 "C13" H 6515 1096 50  0000 L CNN
-F 1 "1u" H 6515 1005 50  0000 L CNN
-F 2 "Swadge_Parts:C_0603_1608Metric" H 6438 900 50  0001 C CNN
-F 3 "" H 6400 1050 50  0001 C CNN
-F 4 "10" H 0   0   50  0001 C CNN "Cost100"
-F 5 "1276-1036-1-ND" H 0   0   50  0001 C CNN "Digikey"
-F 6 "Y" H 0   0   50  0001 C CNN "Substitutable"
-F 7 "0603 Package" H 6400 1050 50  0001 C CNN "Notes"
-	1    6400 1050
-	1    0    0    -1
-$EndComp
-$Comp
 L power:GND #PWR026
 U 1 1 5C3A920C
@@
 Wire Wire Line
 	6250 1350 6250 900
-Connection ~ 6250 900
 $Comp
 L power:GND #PWR025
@@
 Wire Wire Line
 	6900 1350 6900 900
-Connection ~ 6900 900
 $Comp
 L power:GND #PWR028
@@
 F 7 "Y" H 0   0   50  0001 C CNN "Substitutable"
 	1    7550 1650
-	1    0    0    -1
-$EndComp
-$Comp
-L power:+3.3V #PWR030
-U 1 1 5C3A9743
-P 7550 900
-F 0 "#PWR030" H 7550 750 50  0001 C CNN
-F 1 "+3.3V" H 7565 1073 50  0000 C CNN
-F 2 "" H 7550 900 50  0001 C CNN
-F 3 "" H 7550 900 50  0001 C CNN
-	1    7550 900
-	1    0    0    -1
-$EndComp
-$Comp
-L Swadge_Parts:C C15
-U 1 1 5C3A9749
-P 7700 1050
-F 0 "C15" H 7815 1096 50  0000 L CNN
-F 1 "1u" H 7815 1005 50  0000 L CNN
-F 2 "Swadge_Parts:C_0603_1608Metric" H 7738 900 50  0001 C CNN
-F 3 "" H 7700 1050 50  0001 C CNN
-F 4 "10" H 0   0   50  0001 C CNN "Cost100"
-F 5 "1276-1036-1-ND" H 0   0   50  0001 C CNN "Digikey"
-F 6 "Y" H 0   0   50  0001 C CNN "Substitutable"
-F 7 "0603 Package" H 7700 1050 50  0001 C CNN "Notes"
-	1    7700 1050
-	1    0    0    -1
-$EndComp
-$Comp
-L power:GND #PWR032
-U 1 1 5C3A974F
-P 7700 1250
-F 0 "#PWR032" H 7700 1000 50  0001 C CNN
-F 1 "GND" H 7705 1077 50  0000 C CNN
-F 2 "" H 7700 1250 50  0001 C CNN
-F 3 "" H 7700 1250 50  0001 C CNN
-	1    7700 1250
 	1    0    0    -1
 $EndComp
@@
 Wire Wire Line
 	4950 1350 4950 900
-Connection ~ 4950 900
 Wire Wire Line
 	5600 1350 5600 900
 Wire Wire Line
 	5600 900  5750 900
-Connection ~ 5600 900
 Wire Notes Line
 	9350 500  9350 2450
@@
 	1    0    0    -1
 $EndComp
-Connection ~ 4950 5650
 $Comp
 L Swadge_Parts:C C6
@@
 	4900 2650 4900 3350
 Connection ~ 4900 3350
-Connection ~ 4000 3750
 Wire Wire Line
 	4750 3650 4750 3150
@@
 Wire Wire Line
 	4000 3450 4000 3750
-Connection ~ 4000 3150
 Wire Wire Line
 	7550 1350 7550 900
-Connection ~ 7550 900
 Wire Wire Line
 	4950 3450 4300 3450
 Connection ~ 4300 3450
-Connection ~ 9550 1550
-Connection ~ 10050 950
 Wire Wire Line
 	10050 950  10050 1150
@@
 	1000 2700 700  2700
 Wire Wire Line
-	1300 2700 1400 2700
-Connection ~ 1400 2700
-Wire Wire Line
-	1400 2700 1500 2700
-Wire Wire Line
 	1300 2700 1000 2700
 Connection ~ 1300 2700
@@
 	1    0    0    -1
 $EndComp
-Wire Wire Line
-	8800 5800 9000 5800
 Connection ~ 8800 5800
-Connection ~ 9000 5800
-Wire Wire Line
-	9000 5800 9200 5800
 Wire Wire Line
 	8350 5800 8800 5800
@@
 	1    0    0    -1
 $EndComp
-Connection ~ 7050 5700
 Wire Wire Line
 	7050 5700 7400 5700
@@
 Wire Notes Line
 	7800 4950 7800 4800
-Connection ~ 3250 1250
 Wire Wire Line
 	3250 1150 3250 1250
@@
 Wire Wire Line
 	950  1150 950  1250
-Connection ~ 1900 1250
 Wire Wire Line
 	1900 1150 1900 1250
@@
 	850  6100 850  5950
 $Comp
-L power:GND #PWR0102
-U 1 1 5D73519E
-P 11000 1000
-F 0 "#PWR0102" H 11000 750 50  0001 C CNN
-F 1 "GND" H 11005 827 50  0000 C CNN
-F 2 "" H 11000 1000 50  0001 C CNN
-F 3 "" H 11000 1000 50  0001 C CNN
-	1    11000 1000
-	1    0    0    -1
-$EndComp
-$Comp
 L Swadge_Parts:SW_SPDT SW1
 U 1 1 5C3F7306
@@
 Wire Notes Line
 	6850 2500 6850 6500
+Wire Wire Line
+	1300 2700 1500 2700
+Wire Wire Line
+	8800 5800 9200 5800
+$Comp
+L power:+3.3V #PWR030
+U 1 1 5C3A9743
+P 7550 900
+F 0 "#PWR030" H 7550 750 50  0001 C CNN
+F 1 "+3.3V" H 7565 1073 50  0000 C CNN
+F 2 "" H 7550 900 50  0001 C CNN
+F 3 "" H 7550 900 50  0001 C CNN
+	1    7550 900
+	1    0    0    -1
+$EndComp
+$Comp
+L power:GND #PWR0102
+U 1 1 5D73519E
+P 11000 1000
+F 0 "#PWR0102" H 11000 750 50  0001 C CNN
+F 1 "GND" H 11005 827 50  0000 C CNN
+F 2 "" H 11000 1000 50  0001 C CNN
+F 3 "" H 11000 1000 50  0001 C CNN
+	1    11000 1000
+	1    0    0    -1
+$EndComp
+$Comp
+L power:GND #PWR?
+U 1 1 5DB27E5A
+P 7700 1250
+F 0 "#PWR?" H 7700 1000 50  0001 C CNN
+F 1 "GND" H 7705 1077 50  0000 C CNN
+F 2 "" H 7700 1250 50  0001 C CNN
+F 3 "" H 7700 1250 50  0001 C CNN
+	1    7700 1250
+	1    0    0    -1
+$EndComp
 $EndSCHEMATC

Commit message: This routing is bananas
Connections:
- net +3V3: now also C17.1, C18.1, C2.2, R1.1, U1.1 (VCC), U4.7 (VDD)
- net +5V: now also C3.2
Other:
- moved on the sheet: C3
