File: hardware/swadge-barrel-headband/swadge-barrel-headband.kicad_pcb (KiCad board)
At the start: 2 copper layers, 33 x 5 mm, 2 parts

Commit message: Tweaking
Other:
- board text added: "(240) 808-2255"
Changed lines of the file:
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@@
   (general
     (thickness 1.6)
-    (drawings 93)
+    (drawings 95)
     (tracks 0)
     (zones 0)
@@
     (pad 1 thru_hole rect (at 0 0) (size 1 1) (drill 0.65) (layers *.Cu *.Mask))
   )
+  (gr_text "(240) 808-2255" (at 0 0) (layer B.SilkS)
+    (effects (font (size 2 2) (thickness 0.3)) (justify mirror))
+  )
   (gr_poly (pts (xy -11.5 2.249999) (xy -9.648612 2.249999) (xy -9.649 -1.810727) (xy -6.045 -1.810727) (xy -6.045215 2.249999) (xy -1.552466 2.249999) (xy -1.552 -1.810727) (xy 2.050999 -1.810727) (xy 2.050999 2.249999) (xy 6.544698 2.249999) (xy 6.545 -1.81074) (xy 10.148 -1.81074) (xy 10.148096 2.249999) (xy 12 2.249999) (xy 12 1.810999) (xy 10.586999 1.810999) (xy 10.586999 -2.250017) (xy 6.104999 -2.250017) (xy 6.104936 1.810999) (xy 2.491 1.810999) (xy 2.49155 -2.250017) (xy 2.490449 -2.250017) (xy -1.990449 -2.250017) (xy -1.99155 -2.250017) (xy -1.991 1.810999) (xy -5.605998 1.810999) (xy -5.605999 -2.250017) (xy -10.088 -2.25) (xy -10.087896 1.810999) (xy -11.5 1.810999) (xy -11.5 2.249999)) (layer F.Cu) (width 0.163738))
